File: SchematicsAndPCB/Controller.sch (EAGLE design)
At the start: 76 parts, among them J5 DCJ0202, T1 BC237, T10 BC237, T11 BC237, T12 BC237, T13 BC237, T14 BC237, T17 BC237, T18 BC237, T2 BC237, T3 BC237, T4 BC237, T5 BC237, T6 BC237, T7 BC237, T8 BC237, T9 BC237

Commit message: PCB in progress
Parts:
- removed LED6: LA-401AD, led-7-segment:LA-401AD
- removed S1, S2, S3, S4, S5: (no value), switch-omron:10-XX
- added SV5(MENUBUTTON)1: (no value), con-lsta:FE06-1
Connections:
- net GND: now also SV4(FLOORBUTTON).6, SV5(MENUBUTTON)1.6
- net MB1: now also SV5(MENUBUTTON)1.1; no longer S5.S, S5.S1
- net MB2: now also SV5(MENUBUTTON)1.2; no longer S4.S, S4.S1
- net MB3: now also SV5(MENUBUTTON)1.3; no longer S3.S, S3.S1
- net MB4: now also SV5(MENUBUTTON)1.4; no longer S2.S, S2.S1
- net MB5: now also SV5(MENUBUTTON)1.5; no longer S1.S, S1.S1
- net ON_BOARDSS1: no longer LED6.A
- net ON_BOARDSS2: no longer LED6.B
- net ON_BOARDSS3: no longer LED6.C
- net ON_BOARDSS4: no longer LED6.D
- net ON_BOARDSS5: no longer LED6.E
- net ON_BOARDSS6: no longer LED6.F
- net ON_BOARDSS7: no longer LED6.G
- net VCC: no longer LED6.A@1, LED6.A@2, S1.P, S1.P1, S2.P, S2.P1, S3.P, S3.P1, S4.P, S4.P1, S5.P, S5.P1, SV4(FLOORBUTTON).6

Commit message: PCB Draft 1
fully routed
Connections:
- removed net SO8: J2.10, J4.10
- new net N$16: R6.1, SV1.2
- net GND: no longer R6.1, SV1.2
- net SO6: now also J2.9, J4.9
- net SO7: now also J2.10, J4.10; no longer J2.9, J4.9
Changed lines of the file:
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@@
-</segment>
-<segment>
-<wire x1="-147.32" y1="68.58" x2="-152.4" y2="68.58" width="0.1524" layer="91"/>
-<pinref part="SV1" gate="G$1" pin="2"/>
-<pinref part="R6" gate="G$1" pin="1"/>
 </segment>
 <segment>
@@
 </segment>
 <segment>
-<pinref part="J2" gate="1" pin="9"/>
-<wire x1="-104.14" y1="243.84" x2="-111.76" y2="243.84" width="0.1524" layer="91"/>
-<label x="-111.76" y="243.84" size="1.778" layer="95"/>
-</segment>
-<segment>
-<pinref part="J4" gate="1" pin="9"/>
-<wire x1="-22.86" y1="246.38" x2="-30.48" y2="246.38" width="0.1524" layer="91"/>
-<label x="-30.48" y="246.38" size="1.778" layer="95"/>
+<pinref part="J2" gate="1" pin="10"/>
+<wire x1="-104.14" y1="241.3" x2="-111.76" y2="241.3" width="0.1524" layer="91"/>
+<label x="-111.76" y="241.3" size="1.778" layer="95"/>
+</segment>
+<segment>
+<pinref part="J4" gate="1" pin="10"/>
+<wire x1="-22.86" y1="243.84" x2="-30.48" y2="243.84" width="0.1524" layer="91"/>
+<label x="-30.48" y="243.84" size="1.778" layer="95"/>
 </segment>
 </net>
@@
 <junction x="-93.98" y="76.2"/>
 <label x="-91.44" y="73.66" size="1.778" layer="95"/>
+</segment>
+<segment>
+<pinref part="J2" gate="1" pin="9"/>
+<wire x1="-104.14" y1="243.84" x2="-111.76" y2="243.84" width="0.1524" layer="91"/>
+<label x="-111.76" y="243.84" size="1.778" layer="95"/>
+</segment>
+<segment>
+<pinref part="J4" gate="1" pin="9"/>
+<wire x1="-22.86" y1="246.38" x2="-30.48" y2="246.38" width="0.1524" layer="91"/>
+<label x="-30.48" y="246.38" size="1.778" layer="95"/>
 </segment>
 </net>
@@
 </segment>
 </net>
-<net name="SO8" class="0">
-<segment>
-<pinref part="J2" gate="1" pin="10"/>
-<wire x1="-104.14" y1="241.3" x2="-111.76" y2="241.3" width="0.1524" layer="91"/>
-<label x="-111.76" y="241.3" size="1.778" layer="95"/>
-</segment>
-<segment>
-<pinref part="J4" gate="1" pin="10"/>
-<wire x1="-22.86" y1="243.84" x2="-30.48" y2="243.84" width="0.1524" layer="91"/>
-<label x="-30.48" y="243.84" size="1.778" layer="95"/>
-</segment>
-</net>
 <net name="SOFTRST" class="0">
 <segment>
@@
 </segment>
 </net>
+<net name="N$16" class="0">
+<segment>
+<pinref part="SV1" gate="G$1" pin="2"/>
+<pinref part="R6" gate="G$1" pin="1"/>
+<wire x1="-152.4" y1="68.58" x2="-147.32" y2="68.58" width="0.1524" layer="91"/>
+</segment>
+</net>
