File: SchematicsAndPCB/Controller.brd (EAGLE design)
At the start: 100 x 80 mm, 71 parts, among them J5 DCJ0202, T1 BC237, T10 BC237, T11 BC237, T12 BC237, T13 BC237, T14 BC237, T17 BC237, T18 BC237, T2 BC237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

Commit message: PCB in progress
Parts:
- moved T1 12.0 mm to (71.1, 10.2)
- moved R6 10.9 mm to (78.7, 11.4), turned to 180 degrees
- moved R7 6.35 mm to (72.4, 15.2), turned to 0 degrees
- moved J3 2.54 mm to (86.4, 53.3), turned to 270 degrees
- moved J1 1.27 mm to (53.3, 53.3)
- moved J4 1.27 mm to (63.5, 53.3), turned to 270 degrees
Routing:
- net VCC: track 79.8 -> 291.5 mm
- net GND: track 291.4 -> 408.3 mm
- net SLEEP: track 0.00 -> 104.2 mm
- net DIR: track 0.00 -> 98.4 mm
- net DIAGNOSIS: track 0.00 -> 78.5 mm
- net SS7: track 0.00 -> 55.8 mm
- net SS1: track 0.00 -> 53.2 mm
- net SS2: track 0.00 -> 53.2 mm
- net SS6: track 0.00 -> 52.5 mm
- net SS5: track 0.00 -> 52.5 mm
- net SS4: track 0.00 -> 52.5 mm
- net SS3: track 0.00 -> 52.5 mm
- net MOTORCLK: track 0.00 -> 46.6 mm
- net MOTORVCC: track 67.7 -> 114.0 mm
- net SO7: track 0.00 -> 40.2 mm
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
Commit message: PCB Draft 1
fully routed
Parts:
- moved R6 85.8 mm to (8.89, 61.2), turned to 0 degrees
- moved R34 76.5 mm to (90.7, 74.4), turned to 270 degrees
- moved T1 76.4 mm to (11.4, 57.9), turned to 180 degrees
- moved LED4 62.3 mm to (90.7, 68.1), turned to 90 degrees
- moved R7 61.5 mm to (25.1, 54.6), turned to 180 degrees
- moved R29 27.7 mm to (65.0, 16.5), turned to 0 degrees
- moved LED1 26.9 mm to (68.8, 10.9), turned to 180 degrees
- moved R33 25.0 mm to (76.7, 16.8)
- moved LED3 24.9 mm to (80.8, 19.3), turned to 180 degrees
- moved R30 23.7 mm to (65.0, 14.2), turned to 0 degrees
- moved T17 23.0 mm to (61.2, 10.9), turned to 180 degrees
- moved R32 21.1 mm to (65.0, 18.8), turned to 0 degrees
- moved LED2 20.0 mm to (68.8, 6.35), turned to 180 degrees
- moved RN1 15.0 mm to (7.87, 31.8)
- moved RN2 15.0 mm to (7.87, 48.3)
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Connections:
- removed net SO8: J2.10, J4.10
- new net N$16: R6.1, SV1.2
- net GND: no longer R6.1, SV1.2
- net SO6: now also J2.9, J4.9
- net SO7: now also J2.10, J4.10; no longer J2.9, J4.9
Routing:
- net DIAGNOSIS: track 78.5 -> 5.75 mm
- net VCC: track 291.5 -> 237.6 mm
- net SO6: track 4.34 -> 45.6 mm
- net SO8: track 34.1 -> 0.00 mm
- net MOTORVCC: track 114.0 -> 83.2 mm
- net SLEEP: track 104.2 -> 75.1 mm
- net GND: track 408.3 -> 387.3 mm
- net DIR: track 98.4 -> 77.6 mm
- net SO7: track 40.2 -> 56.4 mm
- net N$38: track 4.07 -> 18.7 mm
- net SEN5: track 14.7 -> 4.49 mm
- net SO5: track 44.0 -> 51.7 mm
- net SEN4: track 16.7 -> 9.15 mm
- net N$3: track 9.20 -> 2.54 mm
- net N$15: track 9.12 -> 15.3 mm
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
Commit message: PCB Ver. 1
Parts:
- moved LED1 10.3 mm to (70.6, 21.1)
- moved R30 6.86 mm to (65.0, 21.1)
- moved T17 3.61 mm to (63.5, 13.7)
Routing:
- net GND: track 387.3 -> 345.3 mm
- net VCC: track 237.6 -> 231.1 mm
- net N$36: track 4.29 -> 9.06 mm
- net N$38: track 18.7 -> 15.8 mm
- net N$40: track 4.65 -> 1.78 mm
- net N$35: track 8.02 -> 5.27 mm
- net MOTORVCC: track 83.2 -> 84.1 mm
- added copper zone on layer 1, net GND
- added copper zone on layer 16, net GND
- added copper zone on layer 16, net MOTORVCC
- added copper zone on layer 16, net N$18
- added copper zone on layer 1, net VCC
Other:
- board text added: "TTU ELEVATOR LAB VER. 1"
