File: SchematicsAndPCB/uController_board/microLift.brd (EAGLE design)
At the start: 100 x 80 mm, 44 parts, among them Q1 ARDUINOR3-NOIOREF-NOTEXT, T1 2N2222, T10 2N2222, T11 2N2222, T12 2N2222, T13 2N2222, T2 2N2222, T3 2N2222, T4 2N2222, T5 2N2222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

Commit message: update
Parts:
- moved R18 25.4 mm to (50.8, 45.0)
- moved R21 25.4 mm to (61.2, 20.6)
- moved T13 25.4 mm to (61.2, 29.7)
- moved T4 25.4 mm to (50.8, 11.4)
- moved T5 25.4 mm to (12.7, 11.4)
- moved T6 25.4 mm to (59.7, 11.4)
- moved T9 25.4 mm to (53.1, 37.6)
- moved JP1 25.4 mm to (3.30, 14.0)
- moved JP2 25.4 mm to (3.30, 31.5)
- moved Q1 25.4 mm to (0.00, 0.00)
- moved R1 25.4 mm to (15.2, 12.7)
- moved R10 25.4 mm to (7.87, 7.62)
- moved R11 25.4 mm to (17.8, 15.2)
- moved R13 25.4 mm to (63.8, 45.0)
- moved R14 25.4 mm to (61.0, 45.0)
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Routing:
- net N$13: track 6.47 -> 5.73 mm
- added copper zone on layer 1, net GND
- added copper zone on layer 16, net GND
Other:
- board size 100 x 80 mm -> 68.8 x 53.3 mm

Commit message: update on u-controller board
Routing:
- net GND: track 221.6 -> 205.3 mm
Other:
- board size 68.8 x 53.3 mm -> 68.8 x 53.8 mm
