File: SchematicsAndPCB/FPGA_Controllerboard/Controller.sch (EAGLE design)
At the start: 71 parts, among them J5 DCJ0202, T1 BC237, T10 BC237, T11 BC237, T12 BC237, T13 BC237, T14 BC237, T17 BC237, T18 BC237, T2 BC237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

Commit message: update on PCB
Parts:
- removed LD1117: 22-23-2031, con-molex:22-23-2031
- added IC1: LM1117T-3.3-V, lm1117:LM1117T-3.3-V
- renumbered SV1 to SENSORIN, SV2(MOTOR_DRIVER) to MOTOR_DRIVER, SV3(SEVENSEG) to SEVENSEG, SV4(FLOORBUTTON) to FLOORBUTTON, SV5(MENUBUTTON)1 to MENUBUTTON
Connections:
- net GND: now also IC1.GND; no longer LD1117-3.S
- net MOTORVCC: now also IC1.IN; no longer LD1117-1.S
- net VCC: now also IC1.OUT; no longer LD1117-2.S

Commit message: additional vcc/gnd + holes + heatsink
Parts:
- added JP1, JP2, JP3: (no value), pinhead:PINHD-1X2
- SEVENSEG: device con-lsta:FE08W -> adafruit:PINHD-1X9
Connections:
- net DIR: now also MOTOR_DRIVER.3; no longer MOTOR_DRIVER.2
- net GND: now also JP1.2, JP2.2, JP3.2, MOTOR_DRIVER.6, SEVENSEG.9; no longer SEVENSEG.8
- net MOTORCLK: now also MOTOR_DRIVER.2; no longer MOTOR_DRIVER.4
- net ON_BOARDSS1: now also SEVENSEG.2; no longer SEVENSEG.1
- net ON_BOARDSS2: now also SEVENSEG.3; no longer SEVENSEG.2
- net ON_BOARDSS3: now also SEVENSEG.4; no longer SEVENSEG.3
- net ON_BOARDSS4: now also SEVENSEG.5; no longer SEVENSEG.4
- net ON_BOARDSS5: now also SEVENSEG.6; no longer SEVENSEG.5
- net ON_BOARDSS6: now also SEVENSEG.7; no longer SEVENSEG.6
- net ON_BOARDSS7: now also SEVENSEG.8; no longer SEVENSEG.7
- net SLEEP: now also MOTOR_DRIVER.4; no longer MOTOR_DRIVER.3
- net VCC: now also JP1.1, JP2.1, JP3.1, SEVENSEG.1
